File: hw/megatemp.brd (EAGLE design)
At the start: 44.7 x 49.8 mm, 30 parts, among them U1 STTS751, U2 STTS751, U3 STTS751, U4 STTS751, U5 STTS751, U6 STTS751, U7 STTS751, U8 STTS751

Commit message: Changed a name
Parts:
- renumbered JP1 to J1
Changed lines of the file:
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@@
 <element name="R11" library="resistor" package="R0402" value="22k" x="22.86" y="45.72" rot="R90"/>
 <element name="R12" library="resistor" package="R0402" value="22k" x="27.94" y="45.72" rot="R90"/>
-<element name="JP1" library="pinhead" package="2X16" value="" x="40.64" y="21.59" smashed="yes" rot="R270">
+<element name="J1" library="pinhead" package="2X16" value="" x="40.64" y="21.59" smashed="yes" rot="R270">
 <attribute name="NAME" x="41.91" y="43.561" size="1.27" layer="25" ratio="10" rot="R180"/>
 <attribute name="VALUE" x="36.195" y="41.91" size="1.27" layer="27" rot="R270"/>
@@
 <contactref element="U1" pad="1"/>
 <contactref element="R9" pad="1"/>
-<contactref element="JP1" pad="3"/>
+<contactref element="J1" pad="3"/>
 <wire x1="7.366" y1="45.07" x2="5.334" y2="43.038" width="0.4064" layer="1"/>
 <wire x1="5.334" y1="43.038" x2="5.334" y2="41.148" width="0.4064" layer="1"/>
@@
 <contactref element="U4" pad="6"/>
 <contactref element="R10" pad="1"/>
-<contactref element="JP1" pad="6"/>
+<contactref element="J1" pad="6"/>
 <wire x1="12.446" y1="45.07" x2="14.224" y2="43.292" width="0.4064" layer="1"/>
 <wire x1="14.224" y1="43.292" x2="14.224" y2="41.148" width="0.4064" layer="1"/>
@@
 <contactref element="U6" pad="1"/>
 <contactref element="R11" pad="1"/>
-<contactref element="JP1" pad="28"/>
+<contactref element="J1" pad="28"/>
 <wire x1="22.86" y1="45.07" x2="21.082" y2="43.292" width="0.4064" layer="1"/>
 <wire x1="21.082" y1="43.292" x2="21.082" y2="41.402" width="0.4064" layer="1"/>
@@
 <contactref element="U7" pad="6"/>
 <contactref element="R12" pad="1"/>
-<contactref element="JP1" pad="25"/>
+<contactref element="J1" pad="25"/>
 <wire x1="27.94" y1="45.07" x2="30.48" y2="42.53" width="0.4064" layer="1"/>
 <wire x1="30.48" y1="42.53" x2="30.487809375" y2="41.402053125" width="0.4064" layer="1"/>
@@
 <contactref element="R11" pad="2"/>
 <contactref element="R10" pad="2"/>
-<contactref element="JP1" pad="4"/>
+<contactref element="J1" pad="4"/>
 <wire x1="41.91" y1="38.1" x2="42.418" y2="38.1" width="0.4064" layer="1"/>
 <wire x1="42.418" y1="38.1" x2="43.942" y2="39.624" width="0.4064" layer="1"/>
@@
 <contactref element="U6" pad="5"/>
 <contactref element="U5" pad="5"/>
-<contactref element="JP1" pad="32"/>
-<contactref element="JP1" pad="31"/>
+<contactref element="J1" pad="32"/>
+<contactref element="J1" pad="31"/>
 <polygon width="0.4064" layer="16">
 <vertex x="0" y="0"/>

Commit message: Updated design to a functional schematic
Connections:
- net SCL1: now also J1.1; no longer J1.3
- net SCL2: now also J1.25; no longer J1.28
- net SDA2: now also J1.28; no longer J1.25
Routing:
- net SDA2: track 66.8 -> 69.8 mm
- net SCL2: track 76.6 -> 73.9 mm
- net SCL1: track 98.3 -> 97.2 mm
Changed lines of the file:
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@@
 <contactref element="U1" pad="1"/>
 <contactref element="R9" pad="1"/>
-<contactref element="J1" pad="3"/>
 <wire x1="7.366" y1="45.07" x2="5.334" y2="43.038" width="0.4064" layer="1"/>
 <wire x1="5.334" y1="43.038" x2="5.334" y2="41.148" width="0.4064" layer="1"/>
@@
 <wire x1="9.106" y1="5.73" x2="5.446" y2="5.73" width="0.3048" layer="1"/>
 <wire x1="5.446" y1="5.73" x2="5.334" y2="5.842" width="0.3048" layer="1"/>
-<wire x1="39.37" y1="38.1" x2="38.862" y2="38.1" width="0.3048" layer="16"/>
-<wire x1="38.862" y1="38.1" x2="31.75" y2="45.212" width="0.4064" layer="16"/>
 <wire x1="31.75" y1="45.212" x2="31.75" y2="46.736" width="0.4064" layer="16"/>
 <wire x1="31.75" y1="46.736" x2="30.734" y2="47.752" width="0.4064" layer="16"/>
@@
 <via x="5.334" y="46.482" extent="1-16" drill="0.6"/>
 <wire x1="5.334" y1="46.482" x2="5.334" y2="43.038" width="0.4064" layer="1"/>
+<contactref element="J1" pad="1"/>
+<wire x1="31.75" y1="45.212" x2="36.322" y2="40.64" width="0.4064" layer="16"/>
+<wire x1="36.322" y1="40.64" x2="39.37" y2="40.64" width="0.4064" layer="16"/>
 </signal>
 <signal name="SDA1">
@@
 <contactref element="U6" pad="1"/>
 <contactref element="R11" pad="1"/>
-<contactref element="J1" pad="28"/>
 <wire x1="22.86" y1="45.07" x2="21.082" y2="43.292" width="0.4064" layer="1"/>
 <wire x1="21.082" y1="43.292" x2="21.082" y2="41.402" width="0.4064" layer="1"/>
@@
 <wire x1="24.6" y1="41.29" x2="21.448" y2="41.29" width="0.3048" layer="1"/>
 <wire x1="21.448" y1="41.29" x2="21.082" y2="41.402" width="0.3048" layer="1"/>
-<wire x1="41.91" y1="7.62" x2="41.91" y2="7.874" width="0.3048" layer="16"/>
-<wire x1="41.91" y1="7.874" x2="40.894" y2="8.89" width="0.3048" layer="16"/>
-<wire x1="40.894" y1="8.89" x2="38.1" y2="8.89" width="0.3048" layer="16"/>
-<wire x1="38.1" y1="8.89" x2="33.528" y2="8.89" width="0.4064" layer="16"/>
-<wire x1="33.528" y1="8.89" x2="31.496" y2="6.858" width="0.4064" layer="16"/>
-<wire x1="31.496" y1="6.858" x2="25.146" y2="6.858" width="0.4064" layer="16"/>
+<wire x1="34.544" y1="6.858" x2="25.146" y2="6.858" width="0.4064" layer="16"/>
 <via x="25.146" y="6.858" extent="1-16" drill="0.6"/>
 <wire x1="25.146" y1="6.858" x2="21.336" y2="6.858" width="0.4064" layer="1"/>
 <wire x1="21.336" y1="6.858" x2="21.082" y2="7.112" width="0.4064" layer="1"/>
+<contactref element="J1" pad="25"/>
+<wire x1="34.544" y1="6.858" x2="37.846" y2="10.16" width="0.4064" layer="16"/>
+<wire x1="37.846" y1="10.16" x2="39.37" y2="10.16" width="0.4064" layer="16"/>
 </signal>
 <signal name="SDA2">
@@
 <contactref element="U7" pad="6"/>
 <contactref element="R12" pad="1"/>
-<contactref element="J1" pad="25"/>
 <wire x1="27.94" y1="45.07" x2="30.48" y2="42.53" width="0.4064" layer="1"/>
 <wire x1="30.48" y1="42.53" x2="30.487809375" y2="41.402053125" width="0.4064" layer="1"/>
@@
 <wire x1="30.575753125" y1="28.699146875" x2="30.656603125" y2="17.02098125" width="0.4064" layer="1"/>
 <wire x1="30.656603125" y1="17.02098125" x2="30.70410625" y2="10.15979375" width="0.4064" layer="1"/>
-<wire x1="30.70410625" y1="10.15979375" x2="30.734" y2="5.842" width="0.4064" layer="1"/>
+<wire x1="30.70410625" y1="10.15979375" x2="30.73050625" y2="6.346459375" width="0.4064" layer="1"/>
+<wire x1="30.73050625" y1="6.346459375" x2="30.734" y2="5.842" width="0.4064" layer="1"/>
 <wire x1="26.2" y1="41.29" x2="30.37575625" y2="41.29" width="0.3048" layer="1"/>
 <wire x1="30.37575625" y1="41.29" x2="30.487809375" y2="41.402053125" width="0.3048" layer="1"/>
@@
 <wire x1="26.2" y1="5.73" x2="30.622" y2="5.73" width="0.3048" layer="1"/>
 <wire x1="30.622" y1="5.73" x2="30.734" y2="5.842" width="0.3048" layer="1"/>
-<wire x1="39.37" y1="10.16" x2="30.7043125" y2="10.16" width="0.4064" layer="1"/>
 <wire x1="30.7043125" y1="10.16" x2="30.70410625" y2="10.15979375" width="0.4064" layer="1"/>
+<contactref element="J1" pad="28"/>
+<wire x1="41.91" y1="7.62" x2="40.636459375" y2="6.346459375" width="0.4064" layer="1"/>
+<wire x1="40.636459375" y1="6.346459375" x2="30.73050625" y2="6.346459375" width="0.4064" layer="1"/>
 </signal>
 <signal name="N$2">
